File: KiCad PiHat/Lec18-PCB_kicad.kicad_pcb (KiCad board)
At the start: 2 copper layers, 65 x 56 mm, 27 parts, among them J1 Conn_01x03_Pin, J10 Conn_01x02_Pin, J2 Conn_01x03_Pin, J3 Conn_01x03_Pin, J4 Conn_01x03_Pin, J5 Screw_Terminal_01x02, J6 Conn_01x03_Pin, J7 Conn_01x03_Pin, J8 Conn_01x04_Pin, J9 Conn_01x04_Pin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

Commit message: Fix some minor mistakes with the PCB design.
Parts:
- moved J5 5.08 mm to (81.5, 77.0), turned to 90 degrees
Routing:
- net /GPIO5: track 65.8 -> 59.2 mm, vias 1 -> 3
- net GND: track 229.6 -> 231.4 mm
- net /5V_Ext: track 69.7 -> 68.3 mm
